File: el_pi_hat.sch (KiCad schematic (older format))
At the start: 74 parts, among them J1 12V, J2 UART, J3 Raspberry Pi Header, J4 TRX, J5 MIC, J6 LINE OUT, J7 LINE IN, J8 HP OUT, J9 HP OUT, Q1 2N7002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

Commit message: Dropping 3M32 resistor to 1M4.
The DC/DC converter is currently trimmed to 5.1 V. Since the
Raspberry Pi can take more than that, we increase the voltage
to 5.25 V. This appears to be the recommended operating voltage.

In order to achieve this, a trimming resistor of 1M375 is
required. We use 1M4. Since we also use this resistor value to
dissipate stray charge on FET and microcontroller inputs, those
resistors are dropped in value as well. This is a good thing since
the value was uncomfortably high (and still remains somewhat high
even after the change).

Fixes #2.
Parts:
- R1, R14, R18, R29, R3: value 3M32 -> 1M4
Changed lines of the file:
@@
 P 10200 5200
 F 0 "R29" H 10130 5154 50  0000 R CNN
-F 1 "3M32" H 10130 5245 50  0000 R CNN
+F 1 "1M4" H 10130 5245 50  0000 R CNN
 F 2 "Resistor_SMD:R_0603_1608Metric" V 10130 5200 50  0001 C CNN
 F 3 "~" H 10200 5200 50  0001 C CNN
@@
 P 8850 6000
 F 0 "R18" H 8780 5954 50  0000 R CNN
-F 1 "3M32" H 8780 6045 50  0000 R CNN
+F 1 "1M4" H 8780 6045 50  0000 R CNN
 F 2 "Resistor_SMD:R_0603_1608Metric" V 8780 6000 50  0001 C CNN
 F 3 "~" H 8850 6000 50  0001 C CNN
@@
 P 3600 6900
 F 0 "R1" H 3670 6946 50  0000 L CNN
-F 1 "3M32" H 3670 6855 50  0000 L CNN
+F 1 "1M4" H 3670 6855 50  0000 L CNN
 F 2 "Resistor_SMD:R_0603_1608Metric" V 3530 6900 50  0001 C CNN
 F 3 "~" H 3600 6900 50  0001 C CNN
@@
 P 3850 5450
 F 0 "R3" V 3800 5250 50  0000 C CNN
-F 1 "3M32" V 3850 5450 50  0000 C CNN
+F 1 "1M4" V 3850 5450 50  0000 C CNN
 F 2 "Resistor_SMD:R_0603_1608Metric" V 3780 5450 50  0001 C CNN
 F 3 "~" H 3850 5450 50  0001 C CNN
@@
 P 6850 6100
 F 0 "R14" H 6920 6146 50  0000 L CNN
-F 1 "3M32" H 6920 6055 50  0000 L CNN
+F 1 "1M4" H 6920 6055 50  0000 L CNN
 F 2 "Resistor_SMD:R_0603_1608Metric" V 6780 6100 50  0001 C CNN
 F 3 "~" H 6850 6100 50  0001 C CNN

Commit message: Adding diode to address case where DC/DC converter is reverse biased
The datasheet of the DC/DC converter recommends a (normally) reverse
biased diode across the regulator. This is to prevent damage in case
the output is at a higher voltage than the input.

Since this condition would apply if somebody powers the Raspberry Pi
directly (i.e. not using the hat), it is strongly recommended to add
the diode.

Fixes #1
Parts:
- added D?: B340, Diode_SMD:D_SMC, symbol Device:D
Connections:
- net +12V: now also D?.1 (K)
- net +5V: now also D?.2 (A)
Changed lines of the file:
@@
 I2S_LRCLK
 Wire Wire Line
-	3550 5050 4150 5050
+	3550 5050 3800 5050
 Connection ~ 4150 5050
 $Comp
@@
 Wire Wire Line
 	7250 4000 7450 4000
-Wire Wire Line
-	2250 5050 2650 5050
-Connection ~ 2650 5050
-Wire Wire Line
-	2650 5050 2750 5050
-$Comp
-L power:+12V #PWR09
-U 1 1 5F997767
-P 2650 5050
-F 0 "#PWR09" H 2650 4900 50  0001 C CNN
-F 1 "+12V" H 2665 5223 50  0000 C CNN
-F 2 "" H 2650 5050 50  0001 C CNN
-F 3 "" H 2650 5050 50  0001 C CNN
-	1    2650 5050
-	1    0    0    -1
-$EndComp
 $Comp
 L Device:R R13
@@
 Text Notes 7200 1350 0    50   ~ 0
 FIXME:\nMisplaced on PCB
+$Comp
+L Device:D D?
+U 1 1 5F6CA7B4
+P 3150 4600
+F 0 "D?" H 3350 4550 50  0000 L CNN
+F 1 "B340" H 3350 4450 50  0000 L CNN
+F 2 "Diode_SMD:D_SMC" H 3150 4600 50  0001 C CNN
+F 3 "~" H 3150 4600 50  0001 C CNN
+F 4 "B340-FDICT-ND" V 3150 4600 50  0001 C CNN "DIGIKEY"
+	1    3150 4600
+	1    0    0    -1
+$EndComp
+$Comp
+L power:+12V #PWR09
+U 1 1 5F997767
+P 2650 4600
+F 0 "#PWR09" H 2650 4450 50  0001 C CNN
+F 1 "+12V" H 2665 4773 50  0000 C CNN
+F 2 "" H 2650 4600 50  0001 C CNN
+F 3 "" H 2650 4600 50  0001 C CNN
+	1    2650 4600
+	1    0    0    -1
+$EndComp
+Wire Wire Line
+	3300 4600 3800 4600
+Wire Wire Line
+	3800 4600 3800 5050
+Wire Wire Line
+	2250 5050 2650 5050
+Connection ~ 3800 5050
+Wire Wire Line
+	3800 5050 4150 5050
+Wire Wire Line
+	3000 4600 2650 4600
+Wire Wire Line
+	2650 4600 2650 5050
+Connection ~ 2650 4600
+Connection ~ 2650 5050
+Wire Wire Line
+	2650 5050 2750 5050
 $EndSCHEMATC

Commit message: Adding ability to short out ATtiny chip
In case somebody decides not to use the Quaselsperre PTT timeout
timer watchdog, it would be nice to have a normally unpopulated
resistor that would connect the PTT input to the PTT output.

The documentation was updated accordingly.

Fixes #3.
Parts:
- added R?: NP, Resistor_SMD:R_0603_1608Metric, symbol Device:Jumper_NO_Small
- gave numbers to parts that had none: 1
Connections:
- net PI_PTT: now also R?.2
- net at R17.2, U2.3 (PB1): now also R?.1
Other:
- note added: "Short to\nbypass\nATtiny."
Changed lines of the file:
@@
 	8850 5850 8300 5850
 Wire Wire Line
-	8000 5850 6300 5850
+	8000 5850 7500 5850
 Wire Wire Line
 	6300 5950 6850 5950
-Wire Wire Line
-	8400 5950 8400 6400
-Wire Wire Line
-	8400 6400 10700 6400
 Wire Wire Line
 	5700 5300 5950 5300
@@
 Connection ~ 6850 5950
 Wire Wire Line
-	6850 5950 8400 5950
+	6850 5950 7300 5950
 Wire Wire Line
 	5900 2700 5750 2700
@@
 FIXME:\nMisplaced on PCB
 $Comp
-L Device:D D?
+L Device:D D5
 U 1 1 5F6CA7B4
 P 3150 4600
-F 0 "D?" H 3350 4550 50  0000 L CNN
+F 0 "D5" H 3350 4550 50  0000 L CNN
 F 1 "B340" H 3350 4450 50  0000 L CNN
 F 2 "Diode_SMD:D_SMC" H 3150 4600 50  0001 C CNN
@@
 Wire Wire Line
 	2650 5050 2750 5050
+$Comp
+L Device:Jumper_NO_Small R?
+U 1 1 5F703687
+P 7500 6100
+F 0 "R?" V 7454 6148 50  0000 L CNN
+F 1 "NP" V 7545 6148 50  0000 L CNN
+F 2 "Resistor_SMD:R_0603_1608Metric" H 7500 6100 50  0001 C CNN
+F 3 "~" H 7500 6100 50  0001 C CNN
+	1    7500 6100
+	0    1    1    0
+$EndComp
+Wire Wire Line
+	7300 6400 7300 5950
+Wire Wire Line
+	7300 6400 7500 6400
+Wire Wire Line
+	7500 6000 7500 5850
+Connection ~ 7500 5850
+Wire Wire Line
+	7500 5850 6300 5850
+Wire Wire Line
+	7500 6200 7500 6400
+Connection ~ 7500 6400
+Wire Wire Line
+	7500 6400 10700 6400
+Text Notes 7700 6250 0    50   ~ 0
+Short to\nbypass\nATtiny.
+Wire Notes Line
+	7400 6000 8050 6000
+Wire Notes Line
+	8050 6000 8050 6300
+Wire Notes Line
+	8050 6300 7400 6300
+Wire Notes Line
+	7400 6300 7400 6000
 $EndSCHEMATC

Commit message: Adding "DNP" fields to R2 and R5.
This is to hide them from the BOM. See #6.
Parts:
- R2: DNP (none) -> DNP
- R5: renamed from R?; DNP (none) -> DNP
Changed lines of the file:
@@
 F 2 "Resistor_SMD:R_0603_1608Metric" V 3780 5350 50  0001 C CNN
 F 3 "~" H 3850 5350 50  0001 C CNN
+F 4 "DNP" V 3850 5350 50  0001 C CNN "DNP"
 	1    3850 5350
 	0    1    1    0
@@
 	2650 5050 2750 5050
 $Comp
-L Device:Jumper_NO_Small R?
+L Device:Jumper_NO_Small R5
 U 1 1 5F703687
 P 7500 6100
-F 0 "R?" V 7454 6148 50  0000 L CNN
+F 0 "R5" V 7454 6148 50  0000 L CNN
 F 1 "NP" V 7545 6148 50  0000 L CNN
 F 2 "Resistor_SMD:R_0603_1608Metric" H 7500 6100 50  0001 C CNN
 F 3 "~" H 7500 6100 50  0001 C CNN
+F 4 "DNP" V 7500 6100 50  0001 C CNN "DNP"
 	1    7500 6100
 	0    1    1    0

Commit message: Fixing wrong BOM syntax for DIGIKEY field in U1
"DIGIKEY" was used both in the field name as well as in the value.
Parts:
- U1: DIGIKEY DIGIKEY 945-3252-1-ND‎ -> 945-3252-1-ND‎
Changed lines of the file:
@@
 F 2 "Converter_DCDC:Converter_DCDC_RECOM_RPMx.x-x.0" H 3200 4550 50  0001 C CNN
 F 3 "https://www.recom-power.com/pdf/Innoline/RPM-2.0.pdf" H 3125 5400 50  0001 C CNN
-F 4 "DIGIKEY 945-3252-1-ND‎" H 3150 5350 50  0001 C CNN "DIGIKEY"
+F 4 "945-3252-1-ND‎" H 3150 5350 50  0001 C CNN "DIGIKEY"
 	1    3150 5350
 	1    0    0    -1

Commit message: Bumping Rev. from 1.0 to 1.1 in schematic and PCB
Other:
- note added: "HB9UF EchoLink Hat Rev. 1.1"
- note removed: "HB9UF EchoLink Hat Rev. 1.0"
Changed lines of the file:
@@
 	8850 5600 8850 5500
 Text Notes 600  1000 0    250  ~ 50
-HB9UF EchoLink Hat Rev. 1.0
+HB9UF EchoLink Hat Rev. 1.1
 $Comp
 L Device:R R14
